File: blackbox_rev1/blackbox_rev1.kicad_pcb (KiCad board)
At the start: 2 copper layers, 2 parts, among them U1 Teensy4.1_DEV-16771, U2 OKI

Commit message: Leads helped at CDR
Rearranged board and made edge cuts
Parts:
- removed U2: OKI, MRDT_Devices:OKI_Horizontal
- moved U1 136.1 mm to (136.3, 105.5), turned to 180 degrees
Routing:
- net +3V3: track 0.00 -> 84.4 mm
- net Net-(Conn2-Pad5): track 30.6 -> 6.58 mm, vias 1 -> 0
- net Net-(Conn2-Pad6): track 25.2 -> 6.53 mm, vias 2 -> 0
- net +5V: track 18.4 -> 0.00 mm
- net +3.3VP: track 26.2 -> 44.2 mm, vias 1 -> 0
- net Net-(C3-Pad2): track 49.7 -> 35.4 mm, vias 4 -> 0
- net Net-(Conn2-Pad1): track 22.5 -> 9.85 mm, vias 1 -> 0
- net Net-(Conn2-Pad2): track 22.0 -> 9.85 mm, vias 3 -> 0
- net Net-(C3-Pad1): track 20.0 -> 14.8 mm
- net Net-(Conn2-Pad4): track 20.2 -> 15.9 mm, vias 3 -> 0
- net +12V: track 25.3 -> 27.1 mm, vias 1 -> 0
- net GND: vias 11 -> 1
Other:
- board outline added: 72 x 76.5 mm
