File: blackbox_rev1/blackbox_rev1.sch (KiCad schematic (older format))
At the start: 12 parts

Commit message: BOM updates
Parts:
- gave numbers to parts that had none: 11
Changed lines of the file:
@@
 $EndDescr
 $Comp
-L blackbox_rev1-rescue:Teensy4.1_DEV-16771-MRDT_Shields U?
+L blackbox_rev1-rescue:Teensy4.1_DEV-16771-MRDT_Shields U1
 U 1 1 6160FCF1
 P 3300 3850
-F 0 "U?" H 3300 6017 50  0000 C CNN
+F 0 "U1" H 3300 6017 50  0000 C CNN
 F 1 "Teensy4.1_DEV-16771" H 3300 5926 50  0000 C CNN
 F 2 "MODULE_DEV-16771" H 5400 3550 50  0001 L BNN
@@
 $EndComp
 $Comp
-L MRDT_Connectors:AndersonPP Conn?
+L MRDT_Connectors:AndersonPP Conn1
 U 1 1 61611B14
 P 5150 1700
-F 0 "Conn?" H 5358 2087 60  0000 C CNN
+F 0 "Conn1" H 5358 2087 60  0000 C CNN
 F 1 "AndersonPP" H 5358 1981 60  0000 C CNN
 F 2 "" H 5000 1150 60  0001 C CNN
@@
 $EndComp
 $Comp
-L MRDT_Connectors:AndersonPP Conn?
+L MRDT_Connectors:AndersonPP Conn1
 U 2 1 616122F0
 P 5150 2150
-F 0 "Conn?" H 5358 2537 60  0000 C CNN
+F 0 "Conn1" H 5358 2537 60  0000 C CNN
 F 1 "AndersonPP" H 5358 2431 60  0000 C CNN
 F 2 "" H 5000 1600 60  0001 C CNN
@@
 $EndComp
 $Comp
-L power:GND #PWR?
+L power:GND #PWR0101
 U 1 1 616130AA
 P 5800 1600
-F 0 "#PWR?" H 5800 1350 50  0001 C CNN
+F 0 "#PWR0101" H 5800 1350 50  0001 C CNN
 F 1 "GND" H 5805 1427 50  0000 C CNN
 F 2 "" H 5800 1600 50  0001 C CNN
@@
 	5550 1600 5800 1600
 $Comp
-L power:+12V #PWR?
+L power:+12V #PWR0102
 U 1 1 616159A9
 P 5800 2050
-F 0 "#PWR?" H 5800 1900 50  0001 C CNN
+F 0 "#PWR0102" H 5800 1900 50  0001 C CNN
 F 1 "+12V" H 5815 2223 50  0000 C CNN
 F 2 "" H 5800 2050 50  0001 C CNN
@@
 	5550 2050 5800 2050
 $Comp
-L MRDT_Devices:OKI U?
+L MRDT_Devices:OKI U2
 U 1 1 6161645B
 P 7350 3400
-F 0 "U?" H 7400 3350 60  0001 C CNN
+F 0 "U2" H 7400 3350 60  0001 C CNN
 F 1 "OKI" H 7550 3681 60  0000 C CNN
 F 2 "" H 7150 3300 60  0001 C CNN
@@
 $EndComp
 $Comp
-L Device:C_Small C?
+L Device:C_Small C1
 U 1 1 61616D3F
 P 6850 3500
-F 0 "C?" H 6758 3454 50  0000 R CNN
+F 0 "C1" H 6758 3454 50  0000 R CNN
 F 1 "10 UF" H 6758 3545 50  0000 R CNN
 F 2 "" H 6850 3500 50  0001 C CNN
@@
 $EndComp
 $Comp
-L Device:C_Small C?
+L Device:C_Small C2
 U 1 1 61617AC0
 P 8100 3500
-F 0 "C?" H 8192 3546 50  0000 L CNN
+F 0 "C2" H 8192 3546 50  0000 L CNN
 F 1 "10 UF" H 8192 3455 50  0000 L CNN
 F 2 "" H 8100 3500 50  0001 C CNN
@@
 	6850 3300 6850 3400
 $Comp
-L power:+12V #PWR?
+L power:+12V #PWR0103
 U 1 1 6161886B
 P 7150 2750
-F 0 "#PWR?" H 7150 2600 50  0001 C CNN
+F 0 "#PWR0103" H 7150 2600 50  0001 C CNN
 F 1 "+12V" H 7165 2923 50  0000 C CNN
 F 2 "" H 7150 2750 50  0001 C CNN
@@
 	7550 3800 7550 4050
 $Comp
-L power:GND #PWR?
+L power:GND #PWR0104
 U 1 1 6161CCD3
 P 7550 4050
-F 0 "#PWR?" H 7550 3800 50  0001 C CNN
+F 0 "#PWR0104" H 7550 3800 50  0001 C CNN
 F 1 "GND" H 7555 3877 50  0000 C CNN
 F 2 "" H 7550 4050 50  0001 C CNN
@@
 $EndComp
 $Comp
-L power:+5V #PWR?
+L power:+5V #PWR0105
 U 1 1 6161D57D
 P 7950 2750
-F 0 "#PWR?" H 7950 2600 50  0001 C CNN
+F 0 "#PWR0105" H 7950 2600 50  0001 C CNN
 F 1 "+5V" H 7965 2923 50  0000 C CNN
 F 2 "" H 7950 2750 50  0001 C CNN
@@
 Connection ~ 7950 3300
 $Comp
-L Device:Battery_Cell BT?
+L Device:Battery_Cell BT1
 U 1 1 6161DB77
 P 9500 2100
-F 0 "BT?" H 9618 2196 50  0000 L CNN
+F 0 "BT1" H 9618 2196 50  0000 L CNN
 F 1 "Battery_Cell" H 9618 2105 50  0000 L CNN
 F 2 "" V 9500 2160 50  0001 C CNN
@@
 $EndComp
 $Comp
-L power:+3.3VP #PWR?
+L power:+3.3VP #PWR0106
 U 1 1 6161E1AB
 P 9500 1650
-F 0 "#PWR?" H 9650 1600 50  0001 C CNN
+F 0 "#PWR0106" H 9650 1600 50  0001 C CNN
 F 1 "+3.3VP" H 9515 1823 50  0000 C CNN
 F 2 "" H 9500 1650 50  0001 C CNN
@@
 	9500 1650 9500 1900
 $Comp
-L power:GND #PWR?
+L power:GND #PWR0107
 U 1 1 6161E8FC
 P 9500 2400
-F 0 "#PWR?" H 9500 2150 50  0001 C CNN
+F 0 "#PWR0107" H 9500 2150 50  0001 C CNN
 F 1 "GND" H 9505 2227 50  0000 C CNN
 F 2 "" H 9500 2400 50  0001 C CNN
@@
 	9500 2200 9500 2400
 $Comp
-L Connector:TestPoint TP?
+L Connector:TestPoint TP2
 U 1 1 6161F009
 P 10250 2200
-F 0 "TP?" H 10308 2318 50  0000 L CNN
+F 0 "TP2" H 10308 2318 50  0000 L CNN
 F 1 "vBat" H 10308 2227 50  0000 L CNN
 F 2 "" H 10450 2200 50  0001 C CNN
@@
 $EndComp
 $Comp
-L Connector:TestPoint TP?
+L Connector:TestPoint TP1
 U 1 1 6161FE17
 P 8800 2150
-F 0 "TP?" H 8858 2268 50  0000 L CNN
+F 0 "TP1" H 8858 2268 50  0000 L CNN
 F 1 "Real Time Ground" H 8858 2177 50  0000 L CNN
 F 2 "" H 9000 2150 50  0001 C CNN
@@
 Connection ~ 9500 1900
 $Comp
-L power:+5V #PWR?
+L power:+5V #PWR0108
 U 1 1 61621E58
 P 2300 2300
-F 0 "#PWR?" H 2300 2150 50  0001 C CNN
+F 0 "#PWR0108" H 2300 2150 50  0001 C CNN
 F 1 "+5V" H 2315 2473 50  0000 C CNN
 F 2 "" H 2300 2300 50  0001 C CNN
@@
 	2300 2450 2500 2450
 $Comp
-L power:GND #PWR?
+L power:GND #PWR0109
 U 1 1 616229F2
 P 4550 5650
-F 0 "#PWR?" H 4550 5400 50  0001 C CNN
+F 0 "#PWR0109" H 4550 5400 50  0001 C CNN
 F 1 "GND" H 4555 5477 50  0000 C CNN
 F 2 "" H 4550 5650 50  0001 C CNN
@@
 	4100 5650 4550 5650
 $Comp
-L power:GND #PWR?
+L power:GND #PWR0110
 U 1 1 6162352D
 P 4350 5850
-F 0 "#PWR?" H 4350 5600 50  0001 C CNN
+F 0 "#PWR0110" H 4350 5600 50  0001 C CNN
 F 1 "GND" H 4355 5677 50  0000 C CNN
 F 2 "" H 4350 5850 50  0001 C CNN
@@
 	4350 5750 4350 5850
 $Comp
-L power:+5V #PWR?
+L power:+5V #PWR0111
 U 1 1 616242C9
 P 4200 1900
-F 0 "#PWR?" H 4200 1750 50  0001 C CNN
+F 0 "#PWR0111" H 4200 1750 50  0001 C CNN
 F 1 "+5V" H 4215 2073 50  0000 C CNN
 F 2 "" H 4200 1900 50  0001 C CNN
@@
 $EndComp
 $Comp
-L power:+3.3VP #PWR?
+L power:+3.3VP #PWR0112
 U 1 1 616261D8
 P 4500 2200
-F 0 "#PWR?" H 4650 2150 50  0001 C CNN
+F 0 "#PWR0112" H 4650 2150 50  0001 C CNN
 F 1 "+3.3VP" H 4515 2373 50  0000 C CNN
 F 2 "" H 4500 2200 50  0001 C CNN
@@
 	4500 2250 4500 2200
 $Comp
-L power:+3.3V #PWR?
+L power:+3.3V #PWR0113
 U 1 1 6162722D
 P 4300 1950
-F 0 "#PWR?" H 4300 1800 50  0001 C CNN
+F 0 "#PWR0113" H 4300 1800 50  0001 C CNN
 F 1 "+3.3V" H 4315 2123 50  0000 C CNN
 F 2 "" H 4300 1950 50  0001 C CNN
@@
 NoConn ~ 2500 2750
 $Comp
-L Connector:RJ45_LED_Shielded J?
+L Connector:RJ45_LED_Shielded J1
 U 1 1 6165E12B
 P 9700 4650
-F 0 "J?" V 9654 5180 50  0000 L CNN
+F 0 "J1" V 9654 5180 50  0000 L CNN
 F 1 "RJ45_LED_Shielded" V 9745 5180 50  0000 L CNN
 F 2 "" V 9700 4675 50  0001 C CNN
@@
 $EndComp
 $Comp
-L MRDT_Connectors:Molex_uF_D_06 Conn?
+L MRDT_Connectors:Molex_uF_D_06 Conn2
 U 1 1 6165FE42
 P 10150 5750
-F 0 "Conn?" V 10039 5922 60  0000 R CNN
+F 0 "Conn2" V 10039 5922 60  0000 R CNN
 F 1 "Molex_uF_D_06" V 10145 5922 60  0000 R CNN
 F 2 "MRDT_Connectors:MOLEX_uF_D_06_Horizontal" H 10150 6050 60  0001 C CNN
@@
 	10400 4250 10100 4250
 $Comp
-L Device:C_Small C?
+L Device:C_Small C3
 U 1 1 61667689
 P 10750 5250
-F 0 "C?" H 10842 5296 50  0000 L CNN
+F 0 "C3" H 10842 5296 50  0000 L CNN
 F 1 "C_Small" H 10842 5205 50  0000 L CNN
 F 2 "" H 10750 5250 50  0001 C CNN
@@
 NoConn ~ 9400 4250
 $Comp
-L power:GND #PWR?
+L power:GND #PWR0114
 U 1 1 61674BF6
 P 9000 4750
-F 0 "#PWR?" H 9000 4500 50  0001 C CNN
+F 0 "#PWR0114" H 9000 4500 50  0001 C CNN
 F 1 "GND" H 9005 4577 50  0000 C CNN
 F 2 "" H 9000 4750 50  0001 C CNN

Commit message: Updated Capacitor on the ethernet
Parts:
- removed C3: C_Small, symbol Device:C_Small
- added C?: 0.1 uF, symbol Device:CP1_Small
Connections:
- net at J1.2, J1.5: now also C?.1
- net at Conn2.3, J1.8, J1.9: now also C?.2
Changed lines of the file:
@@
 Wire Wire Line
 	10400 4250 10100 4250
-$Comp
-L Device:C_Small C3
-U 1 1 61667689
-P 10750 5250
-F 0 "C3" H 10842 5296 50  0000 L CNN
-F 1 "C_Small" H 10842 5205 50  0000 L CNN
-F 2 "" H 10750 5250 50  0001 C CNN
-F 3 "~" H 10750 5250 50  0001 C CNN
-	1    10750 5250
-	1    0    0    -1
-$EndComp
 Wire Wire Line
 	10750 5350 10400 5350
@@
 Wire Wire Line
 	9000 4650 9200 4650
+$Comp
+L Device:CP1_Small C?
+U 1 1 616A1606
+P 10750 5250
+F 0 "C?" H 10841 5296 50  0000 L CNN
+F 1 "0.1 uF" H 10841 5205 50  0000 L CNN
+F 2 "" H 10750 5250 50  0001 C CNN
+F 3 "~" H 10750 5250 50  0001 C CNN
+	1    10750 5250
+	1    0    0    -1
+$EndComp
 $EndSCHEMATC

Commit message: Made the footprint
Added all the parts. I did my best?
Parts:
- BT1: footprint (none) -> MRDT_Connectors:CR1220_Battery_Holder
- C1, C2: footprint (none) -> Capacitor_SMD:C_0603_1608Metric_Pad1.08x0.95mm_HandSolder
- C3: renamed from C?; footprint (none) -> Capacitor_SMD:C_0603_1608Metric_Pad1.08x0.95mm_HandSolder
- Conn1: footprint (none) -> MRDT_Connectors:Anderson_2_Horizontal_Side_by_Side
- J1: footprint (none) -> MRDT_Connectors:RJ45_Teensy
- TP1, TP2: footprint (none) -> MountingHole:MountingHole_2.5mm
- U1: footprint MODULE_DEV-16771 -> MRDT_Shields:Teensy_4_1_Vertical
- U2: footprint (none) -> MRDT_Devices:OKI_Horizontal
Changed lines of the file:
@@
 F 0 "U1" H 3300 6017 50  0000 C CNN
 F 1 "Teensy4.1_DEV-16771" H 3300 5926 50  0000 C CNN
-F 2 "MODULE_DEV-16771" H 5400 3550 50  0001 L BNN
+F 2 "MRDT_Shields:Teensy_4_1_Vertical" H 5400 3550 50  0001 L BNN
 F 3 "" H 3300 3850 50  0001 L BNN
 F 4 "Manufacturer recommendations" H 5400 3300 50  0001 L BNN "STANDARD"
@@
 F 0 "Conn1" H 5358 2087 60  0000 C CNN
 F 1 "AndersonPP" H 5358 1981 60  0000 C CNN
-F 2 "" H 5000 1150 60  0001 C CNN
+F 2 "MRDT_Connectors:Anderson_2_Horizontal_Side_by_Side" H 5000 1150 60  0001 C CNN
 F 3 "" H 5000 1150 60  0001 C CNN
 	1    5150 1700
@@
 F 0 "Conn1" H 5358 2537 60  0000 C CNN
 F 1 "AndersonPP" H 5358 2431 60  0000 C CNN
-F 2 "" H 5000 1600 60  0001 C CNN
+F 2 "MRDT_Connectors:Anderson_2_Horizontal_Side_by_Side" H 5000 1600 60  0001 C CNN
 F 3 "" H 5000 1600 60  0001 C CNN
 	2    5150 2150
@@
 F 0 "U2" H 7400 3350 60  0001 C CNN
 F 1 "OKI" H 7550 3681 60  0000 C CNN
-F 2 "" H 7150 3300 60  0001 C CNN
+F 2 "MRDT_Devices:OKI_Horizontal" H 7150 3300 60  0001 C CNN
 F 3 "" H 7150 3300 60  0001 C CNN
 	1    7350 3400
@@
 F 0 "C1" H 6758 3454 50  0000 R CNN
 F 1 "10 UF" H 6758 3545 50  0000 R CNN
-F 2 "" H 6850 3500 50  0001 C CNN
+F 2 "Capacitor_SMD:C_0603_1608Metric_Pad1.08x0.95mm_HandSolder" H 6850 3500 50  0001 C CNN
 F 3 "~" H 6850 3500 50  0001 C CNN
 	1    6850 3500
@@
 F 0 "C2" H 8192 3546 50  0000 L CNN
 F 1 "10 UF" H 8192 3455 50  0000 L CNN
-F 2 "" H 8100 3500 50  0001 C CNN
+F 2 "Capacitor_SMD:C_0603_1608Metric_Pad1.08x0.95mm_HandSolder" H 8100 3500 50  0001 C CNN
 F 3 "~" H 8100 3500 50  0001 C CNN
 	1    8100 3500
@@
 F 0 "BT1" H 9618 2196 50  0000 L CNN
 F 1 "Battery_Cell" H 9618 2105 50  0000 L CNN
-F 2 "" V 9500 2160 50  0001 C CNN
+F 2 "MRDT_Connectors:CR1220_Battery_Holder" V 9500 2160 50  0001 C CNN
 F 3 "~" V 9500 2160 50  0001 C CNN
 	1    9500 2100
@@
 F 0 "TP2" H 10308 2318 50  0000 L CNN
 F 1 "vBat" H 10308 2227 50  0000 L CNN
-F 2 "" H 10450 2200 50  0001 C CNN
+F 2 "MountingHole:MountingHole_2.5mm" H 10450 2200 50  0001 C CNN
 F 3 "~" H 10450 2200 50  0001 C CNN
 	1    10250 2200
@@
 F 0 "TP1" H 8858 2268 50  0000 L CNN
 F 1 "Real Time Ground" H 8858 2177 50  0000 L CNN
-F 2 "" H 9000 2150 50  0001 C CNN
+F 2 "MountingHole:MountingHole_2.5mm" H 9000 2150 50  0001 C CNN
 F 3 "~" H 9000 2150 50  0001 C CNN
 	1    8800 2150
@@
 F 0 "J1" V 9654 5180 50  0000 L CNN
 F 1 "RJ45_LED_Shielded" V 9745 5180 50  0000 L CNN
-F 2 "" V 9700 4675 50  0001 C CNN
+F 2 "MRDT_Connectors:RJ45_Teensy" V 9700 4675 50  0001 C CNN
 F 3 "~" V 9700 4675 50  0001 C CNN
 	1    9700 4650
@@
 	9000 4650 9200 4650
 $Comp
-L Device:CP1_Small C?
+L Device:CP1_Small C3
 U 1 1 616A1606
 P 10750 5250
-F 0 "C?" H 10841 5296 50  0000 L CNN
+F 0 "C3" H 10841 5296 50  0000 L CNN
 F 1 "0.1 uF" H 10841 5205 50  0000 L CNN
-F 2 "" H 10750 5250 50  0001 C CNN
+F 2 "Capacitor_SMD:C_0603_1608Metric_Pad1.08x0.95mm_HandSolder" H 10750 5250 50  0001 C CNN
 F 3 "~" H 10750 5250 50  0001 C CNN
 	1    10750 5250

Commit message: Leads helped at CDR
Rearranged board and made edge cuts
Parts:
- Conn2: footprint MRDT_Connectors:MOLEX_uF_D_06_Horizontal -> Connector_PinSocket_2.00mm:PinSocket_2x03_P2.00mm_Vertical
Connections:
- net +3V3: now also C2.1, U2.3 (Vo)
- removed net +5V: C2.1, U1.5V, U1.VIN, U2.3 (Vo)
- no-connect marks 55 -> 57
Changed lines of the file:
@@
 $EndComp
-$Comp
-L power:+5V #PWR0105
-U 1 1 6161D57D
-P 7950 2750
-F 0 "#PWR0105" H 7950 2600 50  0001 C CNN
-F 1 "+5V" H 7965 2923 50  0000 C CNN
-F 2 "" H 7950 2750 50  0001 C CNN
-F 3 "" H 7950 2750 50  0001 C CNN
-	1    7950 2750
-	1    0    0    -1
-$EndComp
-Wire Wire Line
-	7950 2750 7950 3300
-Connection ~ 7950 3300
 $Comp
 L Device:Battery_Cell BT1
@@
 Connection ~ 9500 1900
 $Comp
-L power:+5V #PWR0108
-U 1 1 61621E58
-P 2300 2300
-F 0 "#PWR0108" H 2300 2150 50  0001 C CNN
-F 1 "+5V" H 2315 2473 50  0000 C CNN
-F 2 "" H 2300 2300 50  0001 C CNN
-F 3 "" H 2300 2300 50  0001 C CNN
-	1    2300 2300
-	1    0    0    -1
-$EndComp
-Wire Wire Line
-	2300 2300 2300 2450
-Wire Wire Line
-	2300 2450 2500 2450
-$Comp
 L power:GND #PWR0109
 U 1 1 616229F2
@@
 	4350 5750 4350 5850
 $Comp
-L power:+5V #PWR0111
-U 1 1 616242C9
-P 4200 1900
-F 0 "#PWR0111" H 4200 1750 50  0001 C CNN
-F 1 "+5V" H 4215 2073 50  0000 C CNN
-F 2 "" H 4200 1900 50  0001 C CNN
-F 3 "" H 4200 1900 50  0001 C CNN
-	1    4200 1900
-	1    0    0    -1
-$EndComp
-$Comp
 L power:+3.3VP #PWR0112
 U 1 1 616261D8
@@
 	1    0    0    -1
 $EndComp
-Wire Wire Line
-	4200 1900 4200 1950
-Wire Wire Line
-	4200 1950 4100 1950
 Wire Wire Line
 	4100 2050 4300 2050
@@
 F 0 "Conn2" V 10039 5922 60  0000 R CNN
 F 1 "Molex_uF_D_06" V 10145 5922 60  0000 R CNN
-F 2 "MRDT_Connectors:MOLEX_uF_D_06_Horizontal" H 10150 6050 60  0001 C CNN
+F 2 "Connector_PinSocket_2.00mm:PinSocket_2x03_P2.00mm_Vertical" H 10150 6050 60  0001 C CNN
 F 3 "" H 10150 6050 60  0001 C CNN
 	1    10150 5750
@@
 	1    0    0    -1
 $EndComp
+Connection ~ 7950 3300
+Wire Wire Line
+	7950 2750 7950 3300
+$Comp
+L power:+3V3 #PWR0105
+U 1 1 619873D0
+P 7950 2750
+F 0 "#PWR0105" H 7950 2600 50  0001 C CNN
+F 1 "+3V3" H 7965 2923 50  0000 C CNN
+F 2 "" H 7950 2750 50  0001 C CNN
+F 3 "" H 7950 2750 50  0001 C CNN
+	1    7950 2750
+	1    0    0    -1
+$EndComp
+NoConn ~ 4100 1950
+NoConn ~ 2500 2450
 $EndSCHEMATC

Commit message: removed rescue library
Parts:
- U1: symbol blackbox_rev1-rescue:Teensy4.1_DEV-16771-MRDT_Shields -> MRDT_Shields:Teensy4.1_DEV-16771
Changed lines of the file:
@@
 $EndDescr
 $Comp
-L blackbox_rev1-rescue:Teensy4.1_DEV-16771-MRDT_Shields U1
+L MRDT_Shields:Teensy4.1_DEV-16771 U1
 U 1 1 6160FCF1
 P 3300 3850
